File: eagle.sch (EAGLE design)
At the start: 11 parts, among them IC1 74HCT245, IC2 74HCT245

Commit message: level 3 design
Parts:
- added C10, C11, C12, C5, C6, C7, C8, C9: 0.1uF, passive:CAP0805
- added IC3, IC4: 74HC14D, 74xx-eu:74HC14D
- added R10, R11, R12, R13, R14, R15, R16, R17, R2, R3, R4, R5, R6, R7, R8, R9: 10K, passive:RESISTOR0805-RES
- added R18, R19, R20, R21, R22, R23, R24, R25: 0, passive:RESISTOR0805-RES
- J1, J2: device SparkFun-Connectors:CONN_08X2 -> SparkFun-Connectors:CONN_08X2_SHROUD
- U$1: value RPI3_HATNO_CF -> RPI3_HATNO_DF; device rpi:RPI3_HATNO_CF -> rpi:RPI3_HATNO_DF
Connections:
- removed net S1: J2.2, U$1.GPIO05
- removed net S2: J2.4, U$1.GPIO06
- removed net S3: J2.6, U$1.GPIO12
- removed net S4: J2.8, U$1.GPIO13
- removed net S5: J2.10, U$1.GPIO19
- removed net S6: J2.12, U$1.GPIO16
- removed net S7: J2.14, U$1.GPIO26
- removed net S8: J2.16, U$1.GPIO20
- new net B1_R: J2.2, R18.1, R2.1, R3.2
- new net B1_S: IC3D.O, R18.2, U$1.GPIO05
- new net B2_R: J2.4, R19.1, R4.1, R5.2
- new net B2_S: IC3E.O, R19.2, U$1.GPIO06
- new net B3_R: J2.6, R20.1, R6.1, R7.2
- new net B3_S: IC3F.O, R20.2, U$1.GPIO12
- new net B4_R: J2.8, R21.1, R8.1, R9.2
- new net B4_S: IC4D.O, R21.2, U$1.GPIO13
- new net B5_R: J2.10, R10.1, R11.2, R22.1
- new net B5_S: IC4E.O, R22.2, U$1.GPIO19
- new net B6_R: J2.12, R12.1, R13.2, R23.1
- new net B6_S: IC4F.O, R23.2, U$1.GPIO16
- new net B7_R: J2.14, R14.1, R15.2, R24.1
- new net B7_S: IC4C.O, R24.2, U$1.GPIO26
- new net B8_R: J2.16, R16.1, R17.2, R25.1
- new net B8_S: IC4B.O, R25.2, U$1.GPIO20
- new net N$1: C5.1, IC3D.I, R2.2
- new net N$2: C6.1, IC3E.I, R4.2
- new net N$3: C7.1, IC3F.I, R6.2
- new net N$4: C8.1, IC4D.I, R8.2
- new net N$5: C9.1, IC4E.I, R10.2
- new net N$6: C10.1, IC4F.I, R12.2
- new net N$7: C11.1, IC4C.I, R14.2
- new net N$8: C12.1, IC4B.I, R16.2
- net +3V3: now also IC3P.VCC, IC4P.VCC, R11.1, R13.1, R15.1, R17.1, R3.1, R5.1, R7.1, R9.1
- net GND: now also C10.2, C11.2, C12.2, C5.2, C6.2, C7.2, C8.2, C9.2, IC3P.GND, IC4P.GND
Other:
- moved on the sheet: C1, C2, C3, C4, IC1, IC2, PWR-1, PWR-2, PWR-3, PWR-4, R1, U$1
